File: hardware/pcb/test-board-rev-a/test-board-rev-a.kicad_pcb (KiCad board)
At the start: 4 copper layers, 120 x 90 mm, 56 parts, among them J1 B7B-XH-A(LF)(SN), J2 5V BENCH IN, J3 SBC LINK, J4 VRX GENERIC, J5 DECODER EVM, J6 SWD, U1 ADS8688AIDBT, U2 STM32G0B1CBT6, U3 TLV75533PDBVR

Commit message: feat(hw): add protected pack reference test option
Parts:
- added F2: 1206L010/60WR DNP, Fuse_1206_3216Metric_Pad1.42x1.75mm_HandSolder, F.Cu at (32.0, 102.0)
- added TP33: BNEG_RAW, TestPoint_Loop_D2.50mm_Drill1.0mm, F.Cu at (39.0, 102.0)
- added TP34: LOCAL_GND, TestPoint_Loop_D2.50mm_Drill1.0mm, F.Cu at (45.0, 102.0)
Other:
- board text added: "F2 B- LINK: DNP / REVIEW"

Commit message: fix(hw): connect pack-negative sense path
Parts:
- added R1: 1K00 0.1%, R_0603_1608Metric_Pad0.98x0.95mm_HandSolder, F.Cu at (42.0, 34.0)
- moved R7 26.7 mm to (68.0, 40.0)
- renumbered R1 to R7
Connections:
- R7 pad 1: TAP1_RAW -> BNEG_RAW
- R7 pad 2: TAP1_SER -> BNEG_SENSE

Commit message: fix(architecture): separate control radio and analog video
Parts:
- J4: value VRX GENERIC -> VRX CVBS ONLY
- J5: value DECODER EVM -> DECODER CVBS ONLY
Connections:
- J4 pad 1: +5V_FUSED -> (no net)
- J4 pad 4: VRX_RSSI -> (no net)
- J4 pad 5: VRX_TX -> (no net)
- J4 pad 6: VRX_RX -> (no net)
- J5 pad 1: +5V_FUSED -> (no net)
- J5 pad 4: I2C_SCL -> (no net)
- J5 pad 5: I2C_SDA -> (no net)
- J5 pad 6: ADC_RESET -> (no net)
Other:
- board text added: "J4/J5: 2 GND 3 CVBS OTHERS NC"
