File: hardware/fpv-hat/fpv-hat.kicad_pcb (KiCad board)
At the start: 4 copper layers, 118.5 x 64.5 mm, 106 parts, among them J1 WAVESHARE 40PIN, J2 SMA EDGE A, J3 SMA EDGE B, J4 BALANCE 2S-6S, J5 AV OUT 3.5MM, Q1 BUZZER DRIVER, SW1 UP, SW2 OK, SW3 DOWN, U1 RSSI COMPARATOR, U2 VIDEO SWITCH, U3 CVBS DECODER, U4 1.8V LDO, U5 ADS1115 0x48, U6 ADS1115 0x49, U7 ADS1115 0x4A, U8 AV BUFFER, Y1 14.31818MHz

Commit message: fix(hw): place both diversity antennas on top edge
Parts:
- moved J2 33.4 mm to (61.4, 67.8), turned to 90 degrees
- moved C25 30.4 mm to (92.0, 104.0)
- moved C26 30.4 mm to (95.0, 100.5)
- moved C27 30.4 mm to (98.0, 100.5)
- moved R29 30.4 mm to (99.0, 104.0)
- moved U8 30.4 mm to (95.0, 104.0)
- moved CRA1 21.5 mm to (65.0, 101.0), turned to 0 degrees
- moved FRA 20.5 mm to (62.0, 101.0), turned to 0 degrees
- moved CRA2 17.4 mm to (68.0, 101.0), turned to 0 degrees
- moved RXA 12.2 mm to (69.0, 84.0), turned to -90 degrees
- moved C1 5.59 mm to (82.0, 77.0)
- moved CIN1 4.00 mm to (122.0, 80.5)
- moved COUT1 4.00 mm to (122.0, 83.5)
- moved FB1 4.00 mm to (115.5, 80.5)
- moved FB2 4.00 mm to (115.5, 83.5)
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Other:
- board text added: "RX A / TOP LEFT"
- board text added: "SMA A TOP LEFT"
- board text removed: "RX A / LEFT"
- board text removed: "SMA A LEFT"
